File: layout/organ.kicad_pcb (KiCad board)
At the start: 2 copper layers, 558.8 x 88.9 mm, 194 parts, among them J1 Screw_Terminal_01x04, J2 Screw_Terminal_01x02, Q1 IRF530N, Q10 IRF530N, Q11 IRF530N, Q12 IRF530N, Q13 IRF530N, Q14 IRF530N, Q15 IRF530N, Q16 IRF530N, Q17 IRF530N, Q18 IRF530N, Q19 IRF530N, Q2 IRF530N, Q20 IRF530N, Q21 IRF530N, Q22 IRF530N, Q23 IRF530N, Q24 IRF530N, Q3 IRF530N, Q4 IRF530N, Q5 IRF530N, Q6 IRF530N, Q7 IRF530N, Q8 IRF530N, Q9 IRF530N, U1 uA7805, U2 H11L1, U3 PIC16F887-IP

Commit message: layout
Other:
- board text added: "+"
- board text added: "1"
- board text added: "12V"
- board text added: "4"
- board text added: "A#3"
- board text added: "A#4"
- board text added: "A3"
- board text added: "A4"
- board text added: "B3"
- board text added: "B4"
- board text added: "C#3"
- board text added: "C#4"
- board text added: "C3"
- board text added: "C4"
- board text added: "D#3"
- board text added: "D#4"
- board text added: "D3"
- board text added: "D4"
- board text added: "E3"
- board text added: "E4"
- board text added: "F#3"
- board text added: "F#4"
- board text added: "F3"
- board text added: "F4"
- board text added: "G#3"
- board text added: "G#4"
- board text added: "G3"
- board text added: "G4"
- board text added: "GND"
- board text added: "PFEIFENORGEL"
- board text added: "POWER"
- board text added: "REV A FRITZ 2026"
